File: rev2/4x4rev2.kicad_pcb (KiCad board)
At the start: 2 copper layers, 188.8 x 128.9 mm, 110 parts, among them J1 Conn_01x03, J10 Conn_01x03, J11 Conn_01x03, J12 Conn_01x03, J13 Conn_01x03, J14 Conn_01x03, J15 Conn_01x03, J16 Conn_01x03, J17 Conn_02x03_Odd_Even, J18 From LiPo, J19 To buck, J2 Conn_01x03, J20 From buck, J3 Conn_01x03, J4 Conn_01x03, J5 Conn_01x03, J6 Conn_01x03, J7 Conn_01x03, J8 Conn_01x03, J9 Conn_01x03, SW1 SW_Push, SW2 SW_Push, SW3 SW_Push, SW4 SW_Push, SW5 Reset, SW6 Boot, U1 TPIC6C595N, U3 ESP32-S3-WROOM-1, U4 TPIC6C595N, U5 CD74HC4067M, U6 CD74HC4067M, U7 L7805

Commit message: rev2 done
rev2 done
Parts:
- removed J19: To buck, Connector_PinHeader_2.54mm:PinHeader_1x02_P2.54mm_Vertical
- removed J20: From buck, Connector_PinHeader_2.54mm:PinHeader_1x02_P2.54mm_Vertical
- added C1: 0.1u, Capacitor_SMD:C_0805_2012Metric, F.Cu at (45.2, 48.3)
- added C2: 0.33u, Capacitor_SMD:C_0805_2012Metric, F.Cu at (45.1, 37.5)
- added J21: Conn_01x03, Connector_PinHeader_2.54mm:PinHeader_1x03_P2.54mm_Vertical, F.Cu at (130.9, 18.7)
- added J22: Conn_01x01, Connector_PinHeader_2.54mm:PinHeader_1x01_P2.54mm_Vertical, F.Cu at (34.4, 58.2)
- added J23: Conn_01x01, Connector_PinHeader_2.54mm:PinHeader_1x01_P2.54mm_Vertical, F.Cu at (57.8, 49.9)
- added J24: Conn_01x01, Connector_PinHeader_2.54mm:PinHeader_1x01_P2.54mm_Vertical, F.Cu at (57.7, 58.5)
- added R41: 5k, Resistor_SMD:R_0805_2012Metric_Pad1.20x1.40mm_HandSolder, F.Cu at (138.0, 85.5)
- added R42: 5k, Resistor_SMD:R_0805_2012Metric_Pad1.20x1.40mm_HandSolder, F.Cu at (93.7, 89.7)
- J17: value Conn_02x03_Odd_Even -> Conn_01x01; footprint Connector_IDC:IDC-Header_2x03_P2.54mm_Vertical -> Connector_PinHeader_2.54mm:PinHeader_1x01_P2.54mm_Vertical
- J18: value From LiPo -> Conn_01x02
- SW5: value Reset -> SW_Push
- SW6: value Boot -> SW_Push
- U5, U6: footprint Package_SO:SOIC-24W_7.5x15.4mm_P1.27mm -> CD74HC4067M:SOIC127P1030X265-24N
- moved J17 101.2 mm to (34.1, 49.8), turned to 0 degrees
- moved C23 0.46 mm to (126.6, 125.2)
Connections:
- J17 pad 1: /EN -> +5V
- U1 pad 8: GND -> Net-(U1-~{G})
- U4 pad 8: GND -> Net-(U4-~{G})
Routing:
- net +3.3V: track 341.2 -> 310.3 mm
- net /EN: track 43.8 -> 14.7 mm
- net GND: track 228.2 -> 211.9 mm, vias 48 -> 49
- net /IO0: track 27.6 -> 11.9 mm
- net /RX: track 14.5 -> 7.06 mm
- net /TX: track 12.9 -> 7.59 mm
- net +5V: track 160.7 -> 164.6 mm
- net +7.4V: track 12.3 -> 16.2 mm
- net Net-(U1-~{G}): track 0.00 -> 3.50 mm
- net Net-(U4-~{G}): track 0.00 -> 2.62 mm
Other:
- board text added: "3.3V"
- board text added: "5V"
- board text added: "BOOT"
- board text added: "From volt reg."
- board text added: "GND"
- board text added: "RESET"
- board text added: "TX RX GND"
- board text added: "To volt reg."
