File: rev2/4x4rev2.kicad_sch (KiCad schematic)
At the start: 110 parts, among them J1 Conn_01x03, J10 Conn_01x03, J11 Conn_01x03, J12 Conn_01x03, J13 Conn_01x03, J14 Conn_01x03, J15 Conn_01x03, J16 Conn_01x03, J17 Conn_02x03_Odd_Even, J18 Conn_01x02, J19 Conn_01x02, J2 Conn_01x03, J20 Conn_01x02, J3 Conn_01x03, J4 Conn_01x03, J5 Conn_01x03, J6 Conn_01x03, J7 Conn_01x03, J8 Conn_01x03, J9 Conn_01x03, SW1 SW_Push, SW2 SW_Push, SW3 SW_Push, SW4 SW_Push, SW5 SW_Push, SW6 SW_Push, U1 TPIC6C595N, U3 ESP32-S3-WROOM-1, U4 TPIC6C595N, U5 CD74HC4067M, U6 CD74HC4067M, U7 L7805

Commit message: rev2 done
rev2 done
Parts:
- removed J17: Conn_02x03_Odd_Even, Connector_IDC:IDC-Header_2x03_P2.54mm_Vertical, symbol Connector_Generic:Conn_02x03_Odd_Even
- removed J19, J20: Conn_01x02, Connector_PinHeader_2.54mm:PinHeader_1x02_P2.54mm_Vertical, symbol Connector_Generic:Conn_01x02
- added C1: 0.1u, Capacitor_SMD:C_0805_2012Metric, symbol Device:C
- added C2: 0.33u, Capacitor_SMD:C_0805_2012Metric, symbol Device:C
- added J17, J22, J23, J24: Conn_01x01, Connector_PinHeader_2.54mm:PinHeader_1x01_P2.54mm_Vertical, symbol Connector_Generic:Conn_01x01
- added J21: Conn_01x03, Connector_PinHeader_2.54mm:PinHeader_1x03_P2.54mm_Vertical, symbol Connector_Generic:Conn_01x03
- added R41, R42: 5k, Resistor_SMD:R_0805_2012Metric_Pad1.20x1.40mm_HandSolder, symbol Device:R
- U5, U6: footprint Package_SO:SOIC-24W_7.5x15.4mm_P1.27mm -> CD74HC4067M:SOIC127P1030X265-24N
Connections:
- net +3.3V: now also J23.1 (Pin_1)
- net +5V: now also C1.1, J17.1 (Pin_1)
- net +7.4V: now also C2.1
- net GND: now also C1.2, C2.2, J21.3 (Pin_3), J22.1 (Pin_1), J24.1 (Pin_1), R41.1, R42.1; no longer U1.8 (~{G}), U4.8 (~{G})
- net RX: now also J21.2 (Pin_2)
- net TX: now also J21.1 (Pin_1)
- new net: R42.2, U1.8 (~{G})
- new net: R41.2, U4.8 (~{G})
Other:
- moved on the sheet: J18, R35, R36, SW5, SW6, U7
